File: UINIO-MCU-STC51.kicad_sch (KiCad schematic)
At the start: 186 parts, among them J1 CON6_2, J10 P1.1, J11 RS485, J12 P1.0, J13 RXD, J14 KEY_Power, J15 TXD, J2 CON8, J3 CON8, J4 LCD_CS, J5 Motor, J6 P1.3, J7 CON8, J8 CON8, J9 P1.2, K1 KEY, K10 KEY, K11 KEY, K12 KEY, K13 KEY, K14 KEY, K15 KEY, K16 KEY, K17 RESET, K2 KEY, K3 KEY, K4 KEY, K5 KEY, K6 KEY, K7 KEY, K8 KEY, K9 KEY, Q1 PNP_9012, Q10 PNP_9012, Q11 PNP_9012, Q12 PNP_9012, Q13 PNP_9012, Q14 PNP_9012, Q15 PNP_9012, Q16 PNP_9012, Q17 PNP_9012, Q18 PNP_9012, Q19 PNP_9012, Q2 PNP_9012, Q20 PNP_9012, Q3 PNP_9012, Q4 PNP_9012, Q5 PNP_9012, Q6 PNP_9012, Q7 PNP_9012, Q8 PNP_9012, Q9 PNP_9012, U1 PCF8591, U10 HS0038, U11 CH340T, U12 MAX485, U2 74HC138, U3 74HC138, U4 74HC245, U5 TL431, U6 DS18B20, U7 24C01, U8 STC89C52, U9 DS1302, Y1 11.0592MHz, Y2 32.768KHz, Y3 12MHz

Commit message: Release UINIO-MCU-STC51 version 0.0.1.
Other:
- company: UinIO.com -> 电子技术博客 UinIO.com
- title: UINIO-STC89C52-EVB -> UINIO-MCU-STC51
